File: pcb/MotionDetectorCamera.sch (EAGLE design)
At the start: 91 parts, among them J1 SOLDER-JUMPER, U1 ICE40HX4K-BG121, U2 TPS6280XYKAR, U3 TPS6280XYKAR, U4 W989D6DBGX6I, U5 TPS63805YFFR, U6 AR0330CS1C12SPKA0, U7 W25Q80EWUXIE, X1 SIT8021AI-J4-18S-12.000000E

Commit message: Safety commit
Parts:
- removed R7: 10k, EagleLibrary:RESISTOR0402
- added R23: 10k, EagleLibrary:RESISTOR0402
Connections:
- removed net 1V8: C1.1, C12.1, C16.1, C17.1, C2.1, C21.1, C22.1, C23.1, C24.1, C26.1, C28.1, C29.1, C34.1, C35.1, C36.1, C37.1, C40.1, C41.1, C8.1, R17.2, R22.2, R5.1, R8.1, R9.2, TC1.7, TP4.SIGNAL, U1E.VCCIO_0_D6, U1E.VCCIO_1_F8, U1E.VCCIO_2_H6, U1E.VCCIO_3_E4, U1E.VCCIO_3_G4, U1E.VCC_SPI_L11, U4A.1_VDD, U4A.1_VDDQ, U4A.2_VDD, U4A.2_VDDQ, U4A.3_VDD, U4A.3_VDDQ, U4A.4_VDDQ, U6G$1.VDD, U6G$1.VDD_IO, U7.VDD, X1.VDD
- removed net N$7: R7.1, U3.EN
- new net 2V8GOOD: R23.1, U3.EN, U5.PG
- new net N$2: C1.1, C12.1, C16.1, C17.1, C2.1, C21.1, C22.1, C23.1, C24.1, C26.1, C28.1, C29.1, C34.1, C35.1, C36.1, C37.1, C40.1, C41.1, C8.1, R17.2, R22.2, R5.1, R8.1, R9.2, TC1.7, TP4.SIGNAL, U1E.VCCIO_0_D6, U1E.VCCIO_1_F8, U1E.VCCIO_2_H6, U1E.VCCIO_3_E4, U1E.VCCIO_3_G4, U1E.VCC_SPI_L11, U4A.1_VDD, U4A.1_VDDQ, U4A.2_VDD, U4A.2_VDDQ, U4A.3_VDD, U4A.3_VDDQ, U4A.4_VDDQ, U6A.VDD, U6A.VDD_IO, U7.VDD, X1.VDD
- net 2V8: now also U6A.VAA, U6A.VAA_PIX, U6A.VDD_MIPI, U6A.VDD_PLL; no longer U6G$1.VAA, U6G$1.VAA_PIX, U6G$1.VDD_MIPI, U6G$1.VDD_PLL
- net CLK12MHZ: now also U6B.EXTCLK; no longer U6G$2.EXTCLK
- net GND: now also U6A.AGND, U6A.DGND, U6B.SADDR, U6B.TEST; no longer U6G$1.AGND, U6G$1.DGND, U6G$2.SADDR, U6G$2.TEST
- net PIX_CLK: now also U6B.PIXCLK; no longer U6G$2.PIXCLK
- net PIX_D0: now also U6B.DOUT0; no longer U6G$2.DOUT0
- net PIX_D1: now also U6B.DOUT1; no longer U6G$2.DOUT1
- net PIX_D10: now also U6B.DOUT10; no longer U6G$2.DOUT10
- net PIX_D11: now also U6B.DOUT11; no longer U6G$2.DOUT11
- net PIX_D2: now also U6B.DOUT2; no longer U6G$2.DOUT2
- net PIX_D3: now also U6B.DOUT3; no longer U6G$2.DOUT3
- net PIX_D4: now also U6B.DOUT4; no longer U6G$2.DOUT4
- net PIX_D5: now also U6B.DOUT5; no longer U6G$2.DOUT5
- net PIX_D6: now also U6B.DOUT6; no longer U6G$2.DOUT6
- net PIX_D7: now also U6B.DOUT7; no longer U6G$2.DOUT7
- net PIX_D8: now also U6B.DOUT8; no longer U6G$2.DOUT8
- net PIX_D9: now also U6B.DOUT9; no longer U6G$2.DOUT9
- net PIX_FV: now also U6B.FRAME_VALID; no longer U6G$2.FRAME_VALID
- net PIX_LV: now also U6B.LINE_VALID; no longer U6G$2.LINE_VALID
- net PIX_RST_: now also U6B.RST_; no longer U6G$2.RST_
- net PIX_SCLK: now also U6B.SCLK; no longer U6G$2.SCLK
- net PIX_SDATA: now also U6B.SDATA; no longer U6G$2.SDATA
- net VDD: now also R23.2; no longer R7.2
Other:
- note added: "Gate 1V8 by 2V8 power-good signal, because the image sensor requires 2V8 be powered before other supplies: "It is critical that VDD_PLL (2V8) is ... powered before or at least at the same time as the [other power supplies, such as VDD / VDD_IO (1V8)].""
- moved on the sheet: C27, R13, R14, R16, TP7

Commit message: Safety commit
Connections:
- removed net N$2: C1.1, C12.1, C16.1, C17.1, C2.1, C21.1, C22.1, C23.1, C24.1, C26.1, C28.1, C29.1, C34.1, C35.1, C36.1, C37.1, C40.1, C41.1, C8.1, R17.2, R22.2, R5.1, R8.1, R9.2, TC1.7, TP4.SIGNAL, U1E.VCCIO_0_D6, U1E.VCCIO_1_F8, U1E.VCCIO_2_H6, U1E.VCCIO_3_E4, U1E.VCCIO_3_G4, U1E.VCC_SPI_L11, U4A.1_VDD, U4A.1_VDDQ, U4A.2_VDD, U4A.2_VDDQ, U4A.3_VDD, U4A.3_VDDQ, U4A.4_VDDQ, U6A.VDD, U6A.VDD_IO, U7.VDD, X1.VDD
- new net 1V8: C1.1, C12.1, C16.1, C17.1, C2.1, C21.1, C22.1, C23.1, C24.1, C26.1, C28.1, C29.1, C34.1, C35.1, C36.1, C37.1, C40.1, C41.1, C8.1, R17.2, R22.2, R5.1, R8.1, R9.2, TC1.7, TP4.SIGNAL, U1E.VCCIO_0_D6, U1E.VCCIO_1_F8, U1E.VCCIO_2_H6, U1E.VCCIO_3_E4, U1E.VCCIO_3_G4, U1E.VCC_SPI_L11, U4A.1_VDD, U4A.1_VDDQ, U4A.2_VDD, U4A.2_VDDQ, U4A.3_VDD, U4A.3_VDDQ, U4A.4_VDDQ, U6G$1.VDD, U6G$1.VDD_IO, U7.VDD, X1.VDD
- net 2V8: now also U6G$1.VAA, U6G$1.VAA_PIX, U6G$1.VDD_MIPI, U6G$1.VDD_PLL; no longer U6A.VAA, U6A.VAA_PIX, U6A.VDD_MIPI, U6A.VDD_PLL
- net CLK12MHZ: now also U6G$2.EXTCLK; no longer U6B.EXTCLK
- net GND: now also U6G$1.AGND, U6G$1.DGND, U6G$2.SADDR, U6G$2.TEST; no longer U6A.AGND, U6A.DGND, U6B.SADDR, U6B.TEST
- net PIX_CLK: now also U6G$2.PIXCLK; no longer U6B.PIXCLK
- net PIX_D0: now also U6G$2.DOUT0; no longer U6B.DOUT0
- net PIX_D1: now also U6G$2.DOUT1; no longer U6B.DOUT1
- net PIX_D10: now also U6G$2.DOUT10; no longer U6B.DOUT10
- net PIX_D11: now also U6G$2.DOUT11; no longer U6B.DOUT11
- net PIX_D2: now also U6G$2.DOUT2; no longer U6B.DOUT2
- net PIX_D3: now also U6G$2.DOUT3; no longer U6B.DOUT3
- net PIX_D4: now also U6G$2.DOUT4; no longer U6B.DOUT4
- net PIX_D5: now also U6G$2.DOUT5; no longer U6B.DOUT5
- net PIX_D6: now also U6G$2.DOUT6; no longer U6B.DOUT6
- net PIX_D7: now also U6G$2.DOUT7; no longer U6B.DOUT7
- net PIX_D8: now also U6G$2.DOUT8; no longer U6B.DOUT8
- net PIX_D9: now also U6G$2.DOUT9; no longer U6B.DOUT9
- net PIX_FV: now also U6G$2.FRAME_VALID; no longer U6B.FRAME_VALID
- net PIX_LV: now also U6G$2.LINE_VALID; no longer U6B.LINE_VALID
- net PIX_RST_: now also U6G$2.RST_; no longer U6B.RST_
- net PIX_SCLK: now also U6G$2.SCLK; no longer U6B.SCLK
- net PIX_SDATA: now also U6G$2.SDATA; no longer U6B.SDATA
Other:
- moved on the sheet: R23
