File: pcb/Programmer.sch (EAGLE design)
At the start: 5 parts, among them J1 MINI-USB-JACK, U1 FT232HQ, U2 SN74AVCH4T245RSVR, X1 SIT8021

Commit message: Progress creating programmer board
Parts:
- added R5: 10k, EagleLibrary:RESISTOR0402
- added U3, U4, U5, U6, U7: SN74LV1T125DCKR, EagleLibrary:SN74LV1T125DCKR
- added U8, U9: SN74LV1T126DCKR, EagleLibrary:SN74LV1T126DCKR
- U2: value SN74AVCH4T245RSVR -> SN74LV1T125DCKR; device EagleLibrary:SN74AVCH4T245RSVR -> EagleLibrary:SN74LV1T125DCKR
Connections:
- removed net N$10: U2.2OE_
- removed net N$12: U2.2DIR
- removed net N$5: U2.2A1
- removed net N$6: U2.2A2
- removed net N$7: U2.2B1
- removed net N$8: U2.2B2
- new net FLASH_MODE: U6.EN_, U7.EN_, U8.EN, U9.EN
- new net FTDI_CDONE: U5.Y
- new net FTDI_CRESET_: U4.A
- new net FTDI_CS_: U3.A
- new net FTDI_SCLK: U2.A
- new net FTDI_SI: U7.Y, U9.Y
- new net FTDI_SO: U6.A, U8.A
- new net ICE_CDONE: R5.2, U5.A
- new net ICE_CRESET_: U4.Y
- new net ICE_CS_: U3.Y
- new net ICE_SCLK: U2.Y
- new net ICE_SI: U6.Y, U9.A
- new net ICE_SO: U7.A, U8.Y
- net 1V8: now also R5.1, U2.VDD, U3.VDD, U4.VDD, U6.VDD, U8.VDD; no longer U2.VCCB
- net 3V3: now also U5.VDD, U7.VDD, U9.VDD; no longer U2.1DIR, U2.VCCA
- net GND: now also U2.EN_, U3.EN_, U3.GND, U4.EN_, U4.GND, U5.EN_, U5.GND, U6.GND, U7.GND, U8.GND, U9.GND; no longer U2.1OE_
- net N$1: now also U1C.ADBUS0; no longer U2.1A1
- net N$2: now also U1C.ADBUS1; no longer U2.1A2
- net N$3: now also U1C.ADBUS2; no longer U2.1B1
- net N$4: now also U1C.ADBUS3; no longer U2.1B2

Commit message: Progress creating programmer board
Connections:
- net ICE_CDONE renamed ICE_PRG_CDONE
- net ICE_CRESET_ renamed ICE_PRG_CRESET_
- net ICE_CS_ renamed ICE_PRG_CS_
- net ICE_SCLK renamed ICE_PRG_CLK
- net ICE_SI renamed ICE_PRG_DI
- net ICE_SO renamed ICE_PRG_DO
- removed net FLASH_MODE: U6.EN_, U7.EN_, U8.EN, U9.EN
- removed net FTDI_CDONE: U5.Y
- removed net FTDI_CRESET_: U4.A
- removed net FTDI_CS_: U3.A
- removed net FTDI_SCLK: U2.A
- removed net FTDI_SI: U7.Y, U9.Y
- removed net FTDI_SO: U6.A, U8.A
- removed net N$1: U1C.ADBUS0
- removed net N$2: U1C.ADBUS1
- removed net N$3: U1C.ADBUS2
- removed net N$4: U1C.ADBUS3
- new net CLK12MHZ: X1.OUT
- new net FTDI_FLASH_MODE: U1C.ADBUS5, U6.EN_, U7.EN_, U8.EN, U9.EN
- new net FTDI_PRG_CDONE: U1C.ADBUS6, U5.Y
- new net FTDI_PRG_CLK: U1C.ADBUS0, U2.A
- new net FTDI_PRG_CRESET_: U1C.ADBUS7, U4.A
- new net FTDI_PRG_CS_: U1C.ADBUS4, U3.A
- new net FTDI_PRG_DI: U1C.ADBUS2, U7.Y, U9.Y
- new net FTDI_PRG_DO: U1C.ADBUS1, U6.A, U8.A
- net 3V3: now also X1.VDD
- net GND: now also X1.EN_, X1.GND
Other:
- note added: "- header for TagConnect cable"
- note added: "Flash Mode"
- note added: "SRAM Mode"
- note removed: "- header for TagConnect cable - DPDT switch (to toggle between programming RAM and flash) - level shifter"
- moved on the sheet: R5

Commit message: Finished with programmer schematic
Parts:
- added C1, C10, C11, C13, C14, C16, C17, C18, C19, C20, C21, C22, C23, C3, C5, C7, C9: 100n, EagleLibrary:CAPACITOR0402
- added C12, C4, C6, C8: 10u, EagleLibrary:CAPACITOR1206
- added C15, C2: 10n, EagleLibrary:CAPACITOR0402
- added FB1, FB2, FB3: FERRITE-BEAD1206, EagleLibrary:FERRITE-BEAD1206
- added H1: WURTH-61201021621, EagleLibrary:WURTH-61201021621
- added R1: 12k, EagleLibrary:RESISTOR0402
- added R2: 10k, EagleLibrary:RESISTOR0402
- added U10: TPD4S012DRYR, EagleLibrary:TPD4S012DRYR
Connections:
- new net 5V: C12.1, C3.1, FB1.P$2, H1.6, U1A.VREGIN
- new net N$1: C2.1, R2.2, U1B.RST_
- new net N$13: H1.9
- new net N$3: C11.1, U1A.VCCA
- new net N$4: R1.1, U1B.REF
- new net N$5: C1.1, U1A.VCORE
- new net USB_D+: J1.D+, U10.D+, U1B.DP
- new net USB_D-: J1.D-, U10.D-, U1B.DM
- new net VBUS: C15.1, FB1.P$1, J1.VCC, U10.VBUS
- new net VPHY: C4.1, C5.1, FB2.P$2, U1A.VPHY
- new net VPLL: C6.1, C7.1, FB3.P$2, U1A.VPLL
- net 1V8: now also C16.1, C17.1, C18.1, C19.1, C20.1, H1.7
- net 3V3: now also C10.1, C13.1, C14.1, C21.1, C22.1, C23.1, C8.1, C9.1, FB2.P$1, FB3.P$1, R2.1, U1A.VCCD, U1A.VCCIO
- net CLK12MHZ: now also U1B.OCSI
- net GND: now also C1.2, C10.2, C11.2, C12.2, C13.2, C14.2, C15.2, C16.2, C17.2, C18.2, C19.2, C2.2, C20.2, C21.2, C22.2, C23.2, C3.2, C4.2, C5.2, C6.2, C7.2, C8.2, C9.2, H1.8, J1.GND, R1.2, U10.GND, U1A.AGND, U1A.GND, U1B.TEST
- net ICE_PRG_CDONE: now also H1.5
- net ICE_PRG_CLK: now also H1.2
- net ICE_PRG_CRESET_: now also H1.10
- net ICE_PRG_CS_: now also H1.3
- net ICE_PRG_DI: now also H1.1
- net ICE_PRG_DO: now also H1.4
Other:
- note added: ""OSCO should be left unconnected""
- note added: "FTDI"
- note added: "Header"
- note added: "Level Shifting"
- note added: "USB Jack, ESD Protection"
- note added: "VCCD"
- note added: "VCCIO"
- note added: "VREGIN"
- note removed: "- header for TagConnect cable"
- moved on the sheet: C26, J1, R5, U1A, U1B, U1C, U2, U3, U4, U5, U6, U7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

Commit message: Programmer board progress. Trying to decide whether we can reliably support UART...
Parts:
- added C24: 100n, EagleLibrary:CAPACITOR0402
- added TP1, TP2, TP3: TEST-POINT, EagleLibrary:TEST-POINT
- added U11: SN74LV1T125DCKR, EagleLibrary:SN74LV1T125DCKR
- U8, U9: value SN74LV1T126DCKR -> SN74LV1T125DCKR; device EagleLibrary:SN74LV1T126DCKR -> EagleLibrary:SN74LV1T125DCKR
Connections:
- removed net FTDI_FLASH_MODE: U1C.ADBUS5, U6.EN_, U7.EN_, U8.EN, U9.EN
- new net FTDI_FLASH_EN_: U1C.ACBUS1, U8.EN_, U9.EN_
- new net FTDI_SRAM_EN_: U1C.ACBUS0, U6.EN_, U7.EN_
- new net FTDI_UART_EN_: U11.EN_, U1C.ACBUS2
- net 3V3: now also C24.1, TP3.X, U11.VDD
- net 5V: now also TP2.X
- net CLK12MHZ: now also TP1.X
- net FTDI_PRG_DO: now also U11.Y
- net GND: now also C24.2, U11.GND
- net ICE_PRG_DO: now also U11.A
Other:
- note added: "UART Mode"
- moved on the sheet: C20, C23, H1, U8, U9

Commit message: Commit before switching to 74LV1T126
Parts:
- removed C24: 100n, EagleLibrary:CAPACITOR0402
- removed U11: SN74LV1T125DCKR, EagleLibrary:SN74LV1T125DCKR
- added H2: HEADER-1X3, EagleLibrary:HEADER-1X3
- U8, U9: value SN74LV1T125DCKR -> SN74LV1T126DCKR; device EagleLibrary:SN74LV1T125DCKR -> EagleLibrary:SN74LV1T126DCKR
Connections:
- net FTDI_PRG_CRESET_ renamed FTDI_PRG_CRST_
- net ICE_PRG_CRESET_ renamed ICE_PRG_CRST_
- removed net FTDI_FLASH_EN_: U1C.ACBUS1, U8.EN_, U9.EN_
- removed net FTDI_SRAM_EN_: U1C.ACBUS0, U6.EN_, U7.EN_
- removed net FTDI_UART_EN_: U11.EN_, U1C.ACBUS2
- new net FTDI_FLASH_MODE: U1C.ACBUS0, U6.EN_, U7.EN_, U8.EN, U9.EN
- net 3V3: no longer C24.1, U11.VDD
- net FTDI_PRG_DI: now also H2.2
- net FTDI_PRG_DO: now also H2.1; no longer U11.Y
- net GND: now also H2.3; no longer C24.2, U11.GND
- net ICE_PRG_DO: no longer U11.A
Other:
- note added: "Headers"
- note added: "TagConnect Programmer Cable"
- note added: "UART"
- note removed: "Header"
- note removed: "UART Mode"
- moved on the sheet: C16, C17, C18, C19, C20, C21, C22, C23, H1, R5, U2, U3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

Commit message: Programmer: renumber components
Parts:
- removed C26: 10n, EagleLibrary:CAPACITOR0402
- added C24: 100n, EagleLibrary:CAPACITOR0402
- C1, C16: value 100n -> 10n; PN GRM155R61H104KE19D -> GCM155R71H103JA55D
- C12, C4, C8: value 10u -> 100n; device EagleLibrary:CAPACITOR1206 -> EagleLibrary:CAPACITOR0402; PN GCM31CC71E106KA03K -> GRM155R61H104KE19D
- C2: value 10n -> 10u; device EagleLibrary:CAPACITOR0402 -> EagleLibrary:CAPACITOR1206; PN GCM155R71H103JA55D -> GCM31CC71E106KA03K
- C3, C5: value 100n -> 10u; device EagleLibrary:CAPACITOR0402 -> EagleLibrary:CAPACITOR1206; PN GRM155R61H104KE19D -> GCM31CC71E106KA03K
- R1: value 12k -> 10k; PN CRCW040212K0FKEDC -> CRCW040210K0FKEDC
- R2: value 10k -> 12k; PN CRCW040210K0FKEDC -> CRCW040212K0FKEDC
- U1: value FT232HQ -> TPD4S012DRYR; device EagleLibrary:FT232HQ -> EagleLibrary:TPD4S012DRYR
- U10: value TPD4S012DRYR -> SN74LV1T126DCKR; device EagleLibrary:TPD4S012DRYR -> EagleLibrary:SN74LV1T126DCKR
- U2: value SN74LV1T125DCKR -> FT232HQ; device EagleLibrary:SN74LV1T125DCKR -> EagleLibrary:FT232HQ
- U8: value SN74LV1T126DCKR -> SN74LV1T125DCKR; device EagleLibrary:SN74LV1T126DCKR -> EagleLibrary:SN74LV1T125DCKR
- renumbered R5 to R3
Connections:
- net 1V8: now also C23.1, U5.VDD, U9.VDD; no longer C16.1, U2.VDD, U8.VDD
- net 3V3: now also C12.1, C16.1, C24.1, C3.1, C4.1, R1.1, U10.VDD, U2A.VCCD, U2A.VCCIO, U8.VDD; no longer C10.1, C13.1, C14.1, C23.1, C26.1, R2.1, U1A.VCCD, U1A.VCCIO, U5.VDD, U9.VDD
- net 5V: now also C2.1, C7.1, U2A.VREGIN; no longer C12.1, C3.1, U1A.VREGIN
- net CLK12MHZ: now also U2B.OCSI; no longer U1B.OCSI
- net FTDI_FLASH_MODE: now also U10.EN, U2C.ACBUS0, U4.EN_; no longer U1C.ACBUS0, U6.EN_, U8.EN
- net FTDI_PRG_CDONE: now also U2C.ADBUS6, U8.Y; no longer U1C.ADBUS6, U5.Y
- net FTDI_PRG_CLK: now also U2C.ADBUS0, U3.A; no longer U1C.ADBUS0, U2.A
- net FTDI_PRG_CRST_: now also U2C.ADBUS7, U6.A; no longer U1C.ADBUS7, U4.A
- net FTDI_PRG_CS_: now also U2C.ADBUS4, U5.A; no longer U1C.ADBUS4, U3.A
- net FTDI_PRG_DI: now also U10.Y, U2C.ADBUS2; no longer U1C.ADBUS2, U9.Y
- net FTDI_PRG_DO: now also U2C.ADBUS1, U4.A, U9.A; no longer U1C.ADBUS1, U6.A, U8.A
- net GND: now also C24.2, R2.2, U1.GND, U2A.AGND, U2A.GND, U2B.TEST, U6.EN_, U8.EN_; no longer C26.2, R1.2, U1A.AGND, U1A.GND, U1B.TEST, U2.EN_, U2.GND, U4.EN_
- net ICE_PRG_CDONE: now also U8.A; no longer U5.A
- net ICE_PRG_CLK: now also U3.Y; no longer U2.Y
- net ICE_PRG_CRST_: now also U6.Y; no longer U4.Y
- net ICE_PRG_CS_: now also U5.Y; no longer U3.Y
- net ICE_PRG_DI: now also U10.A, U4.Y; no longer U6.Y, U9.A
- net ICE_PRG_DO: now also U9.Y; no longer U8.Y
- net N$1: now also C15.1, R1.2, U2B.RST_; no longer C2.1, R2.2, U1B.RST_
- net N$3: now also C13.1, U2A.VCCA; no longer C11.1, U1A.VCCA
- net N$4: now also R2.1, U2B.REF; no longer R1.1, U1B.REF
- net N$5: now also C14.1, U2A.VCORE; no longer C1.1, U1A.VCORE
- net USB_D+: now also U1.D+, U2B.DP; no longer U10.D+, U1B.DP
- net USB_D-: now also U1.D-, U2B.DM; no longer U10.D-, U1B.DM
- net VBUS: now also C1.1, U1.VBUS; no longer C15.1, U10.VBUS
- net VPHY: now also C10.1, U2A.VPHY; no longer C4.1, U1A.VPHY
- net VPLL: now also C11.1, U2A.VPLL; no longer C7.1, U1A.VPLL
Other:
- moved on the sheet: C1, C10, C11, C12, C13, C14, C15, C16, C17, C18, C19, C2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

Commit message: Programmer: Update part numbers
Parts:
- H2: MFG (none) -> Molex; PN (none) -> 22-28-4100
Changed lines of the file:
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@@
 <part name="TP2" library="EagleLibrary" deviceset="TEST-POINT" device=""/>
 <part name="TP3" library="EagleLibrary" deviceset="TEST-POINT" device=""/>
-<part name="H2" library="EagleLibrary" deviceset="HEADER-1X3" device="" package3d_urn="urn:adsk.eagle:package:19124821/1"/>
+<part name="H2" library="EagleLibrary" deviceset="HEADER-1X3" device="" package3d_urn="urn:adsk.eagle:package:19124821/1">
+<attribute name="MFG" value="Molex"/>
+<attribute name="PN" value="22-28-4100"/>
+</part>
 </parts>
 <sheets>
@@
 <instance part="H2" gate="G$1" x="393.7" y="10.16" smashed="yes">
 <attribute name="NAME" x="393.7" y="10.922" size="1.778" layer="95"/>
+<attribute name="MFG" x="393.7" y="10.16" size="1.778" layer="96" display="off"/>
+<attribute name="PN" x="393.7" y="10.16" size="1.778" layer="96" display="off"/>
 </instance>
 </instances>
