File: pcb/Programmer.sch (EAGLE design)
At the start: 47 parts, among them J1 MINI-USB-JACK, U1 TPD4S012DRYR, U10 SN74LV1T126DCKR, U2 FT232HQ, U3 SN74LV1T125DCKR, U4 SN74LV1T125DCKR, U5 SN74LV1T125DCKR, U6 SN74LV1T125DCKR, U7 SN74LV1T125DCKR, U8 SN74LV1T125DCKR, U9 SN74LV1T126DCKR, X1 SIT8021

Commit message: Progress
Parts:
- X1: value SIT8021 -> SITIME-SIT8021; device EagleLibrary:SIT8021 -> EagleLibrary:SITIME-SIT8021
Other:
- moved on the sheet: C15, R1, R2, U1, U2B, U2C
