File: pcb/Programmer.brd (EAGLE design)
At the start: 38.1 x 26 mm, 47 parts, among them J1 MINI-USB-JACK, U1 TPD4S012DRYR, U10 SN74LV1T126DCKR, U2 FT232HQ, U3 SN74LV1T125DCKR, U4 SN74LV1T125DCKR, U5 SN74LV1T125DCKR, U6 SN74LV1T125DCKR, U7 SN74LV1T125DCKR, U8 SN74LV1T125DCKR, U9 SN74LV1T126DCKR, X1 SIT8021

Commit message: Progress
Parts:
- J1: device EagleLibrary:AMPHENOLFCI-10033526-N3212MLF -> EagleLibrary:AMPHENOLFCI-10033526-N3222MLF
- X1: value SIT8021 -> SITIME-SIT8021; device EagleLibrary:SIT8021 -> EagleLibrary:SITIME-SIT8021
Changed lines of the file:
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@@
 <?xml version="1.0" encoding="utf-8"?>
 <!DOCTYPE eagle SYSTEM "eagle.dtd">
-<eagle version="9.5.2">
+<eagle version="9.6.2">
 <drawing>
 <settings>
@@
 <attribute name="PN" value="FT232HQ-REEL" x="35.4076" y="5.842" size="1.778" layer="27" display="off"/>
 </element>
-<element name="X1" library="EagleLibrary" package="SIT8021" value="SIT8021" x="13.208" y="18.542" smashed="yes">
+<element name="X1" library="EagleLibrary" package="SITIME-SIT8021" value="SITIME-SIT8021" x="13.208" y="18.542" smashed="yes">
 <attribute name="MFG" value="SiTime" x="13.208" y="18.542" size="1.778" layer="27" display="off"/>
 <attribute name="NAME" x="12.7796" y="19.5756" size="0.508" layer="25" font="vector"/>
@@
 <attribute name="PN" value="GCM155R71H103JA55D" x="14.1732" y="18.542" size="1.778" layer="27" rot="R90" display="off"/>
 </element>
-<element name="J1" library="EagleLibrary" package="AMPHENOLFCI-10033526-N3212MLF" value="MINI-USB-JACK" x="5.461" y="13.081" smashed="yes" rot="R270">
+<element name="J1" library="EagleLibrary" package="AMPHENOLFCI-10033526-N3222MLF" value="MINI-USB-JACK" x="5.461" y="13.081" smashed="yes" rot="R270">
 <attribute name="MFG" value="Amphenol FCI" x="5.461" y="13.081" size="1.778" layer="27" rot="R270" display="off"/>
 <attribute name="NAME" x="4.7181" y="17.1168" size="1.27" layer="25" font="vector"/>
-<attribute name="PN" value="10033526-N3212MLF" x="5.461" y="13.081" size="1.778" layer="27" rot="R270" display="off"/>
+<attribute name="PN" value="10033526-N3222MLF" x="5.461" y="13.081" size="1.778" layer="27" rot="R270" display="off"/>
 </element>
 <element name="U3" library="EagleLibrary" package="SN74LV1T12XDCKR" package3d_urn="urn:adsk.eagle:package:19104715/1" value="SN74LV1T125DCKR" x="28.4988" y="5.671" smashed="yes" rot="MR90">
@@
 <wire x1="19.4811" y1="17.5514" x2="19.6088" y2="17.6791" width="0.2032" layer="16"/>
 <wire x1="19.6088" y1="17.6791" x2="19.6088" y2="18.2398" width="0.2032" layer="16"/>
+<wire x1="19.759" y1="16.0782" x2="22.5044" y2="14.0201" width="0" layer="19" extent="1-16"/>
+<wire x1="16.0521" y1="18.3388" x2="19.3776" y2="17.3376" width="0" layer="19" extent="1-1"/>
+<wire x1="14.1732" y1="18.1095" x2="16.0521" y2="18.3388" width="0" layer="19" extent="1-1"/>
+<wire x1="8.9132" y1="18.923" x2="13.413" y2="18.042" width="0" layer="19" extent="1-16"/>
+<wire x1="20.3776" y1="9.5864" x2="22.5044" y2="14.0201" width="0" layer="19" extent="1-1"/>
+<wire x1="19.9898" y1="6.9603" x2="20.3454" y2="8.7376" width="0" layer="19" extent="1-1"/>
+<wire x1="16.749" y1="6.9313" x2="19.304" y2="6.9603" width="0" layer="19" extent="1-1"/>
+<wire x1="13.6248" y1="6.9313" x2="15.8496" y2="6.9603" width="0" layer="19" extent="1-1"/>
+<wire x1="13.1318" y1="9.8813" x2="12.8781" y2="7.6708" width="0" layer="19" extent="1-1"/>
+<wire x1="8.964" y1="7.1882" x2="12.7254" y2="6.9603" width="0" layer="19" extent="1-1"/>
 </signal>
 <signal name="GND">
@@
 <via x="2.5146" y="20.2184" extent="1-16" drill="0.254"/>
 <via x="30.607" y="24.3078" extent="1-16" drill="0.254"/>
+<wire x1="27.5336" y1="16.9919" x2="30.607" y2="24.3078" width="0" layer="19" extent="16-16"/>
+<wire x1="29.1614" y1="16.136" x2="27.5336" y2="16.2814" width="0" layer="19" extent="1-1"/>
+<wire x1="22.7098" y1="16.0782" x2="25.3342" y2="15.9541" width="0" layer="19" extent="16-16"/>
+<wire x1="20.9804" y1="16.8148" x2="21.5032" y2="16.7386" width="0" layer="19" extent="1-1"/>
+<wire x1="22.5044" y1="16.6631" x2="22.7098" y2="16.0782" width="0" layer="19" extent="1-16"/>
+<wire x1="14.8776" y1="17.3376" x2="14.2748" y2="16.8148" width="0" layer="19" extent="1-1"/>
+<wire x1="21.9717" y1="18.8214" x2="21.9717" y2="17.9578" width="0" layer="19" extent="1-1"/>
+<wire x1="21.9209" y1="9.6774" x2="20.9804" y2="10.1092" width="0" layer="19" extent="1-1"/>
+<wire x1="14.1732" y1="18.9745" x2="14.8776" y2="18.1864" width="0" layer="19" extent="1-1"/>
+<wire x1="13.8176" y1="9.0163" x2="14.2748" y2="10.1092" width="0" layer="19" extent="1-1"/>
+<wire x1="19.8776" y1="9.5864" x2="20.9804" y2="10.1092" width="0" layer="19" extent="1-1"/>
+<wire x1="13.752" y1="11.212" x2="14.2748" y2="10.1092" width="0" layer="19" extent="1-1"/>
+<wire x1="20.3708" y1="18.8976" x2="20.3461" y2="17.5514" width="0" layer="19" extent="16-16"/>
+<wire x1="21.9986" y1="20.3708" x2="21.9717" y2="18.8214" width="0" layer="19" extent="1-1"/>
+<wire x1="11.3277" y1="12.0396" x2="12.9032" y2="11.712" width="0" layer="19" extent="16-16"/>
+<wire x1="16.9171" y1="18.3388" x2="15.3776" y2="17.3376" width="0" layer="19" extent="1-1"/>
+<wire x1="17.8776" y1="18.1864" x2="16.9171" y2="18.3388" width="0" layer="19" extent="1-1"/>
+<wire x1="9.6774" y1="14.3256" x2="11.303" y2="13.3851" width="0" layer="19" extent="16-16"/>
+<wire x1="10.033" y1="15.9519" x2="9.6774" y2="14.3256" width="0" layer="19" extent="1-1"/>
+<wire x1="10.8966" y1="16.129" x2="10.033" y2="15.9519" width="0" layer="19" extent="1-1"/>
+<wire x1="8.186" y1="17.531" x2="8.9132" y2="16.8402" width="0" layer="19" extent="1-16"/>
+<wire x1="12.9032" y1="14.7628" x2="11.2769" y2="15.367" width="0" layer="19" extent="16-16"/>
+<wire x1="9.906" y1="10.5664" x2="11.3277" y2="12.0396" width="0" layer="19" extent="16-16"/>
+<wire x1="8.311" y1="11.481" x2="8.964" y2="10.5664" width="0" layer="19" extent="1-16"/>
+<wire x1="8.186" y1="8.631" x2="8.964" y2="10.5664" width="0" layer="19" extent="1-16"/>
+<wire x1="4.3434" y1="8.631" x2="6.5532" y2="8.631" width="0" layer="19" extent="1-1"/>
+<wire x1="4.3434" y1="17.531" x2="6.5786" y2="17.531" width="0" layer="19" extent="1-1"/>
+<wire x1="19.9898" y1="6.0953" x2="19.6998" y2="8.763" width="0" layer="19" extent="1-1"/>
+<wire x1="18.049" y1="5.0067" x2="19.9898" y2="5.3848" width="0" layer="19" extent="1-1"/>
+<wire x1="14.9248" y1="5.0067" x2="15.8496" y2="5.3848" width="0" layer="19" extent="1-1"/>
+<wire x1="2.5146" y1="20.2184" x2="2.736" y2="17.531" width="0" layer="19" extent="1-1"/>
+<wire x1="25.512" y1="8.2341" x2="21.9209" y2="8.9916" width="0" layer="19" extent="1-16"/>
+<wire x1="30.0482" y1="5.7397" x2="27.7114" y2="8.5344" width="0" layer="19" extent="16-16"/>
+<wire x1="31.7096" y1="4.7087" x2="30.0355" y2="5.0038" width="0" layer="19" extent="16-16"/>
+<wire x1="33.894" y1="9.1231" x2="33.909" y2="5.7143" width="0" layer="19" extent="16-16"/>
+<wire x1="4.2164" y1="4.2926" x2="4.3434" y2="8.631" width="0" layer="19" extent="1-1"/>
 </signal>
 <signal name="1V8">
@@
 <wire x1="36.0934" y1="11.0751" x2="36.0934" y2="11.811" width="0.2032" layer="16"/>
 <via x="36.0934" y="11.811" extent="1-16" drill="0.254"/>
+<wire x1="28.2448" y1="17.8569" x2="31.7014" y2="16.136" width="0" layer="19" extent="1-1"/>
+<wire x1="36.0934" y1="11.811" x2="31.7014" y2="16.136" width="0" layer="19" extent="1-1"/>
+<wire x1="33.909" y1="7.2898" x2="35.194" y2="11.0477" width="0" layer="19" extent="16-16"/>
+<wire x1="30.734" y1="6.6047" x2="33.0096" y2="6.6333" width="0" layer="19" extent="16-16"/>
+<wire x1="28.3972" y1="10.1099" x2="29.1488" y2="6.6333" width="0" layer="19" extent="16-16"/>
+<wire x1="23.114" y1="6.35" x2="26.812" y2="10.1587" width="0" layer="19" extent="16-16"/>
 </signal>
 <signal name="FTDI_PRG_CLK">
@@
 <wire x1="18.8214" y1="18.8214" x2="18.8214" y2="18.415" width="0.2032" layer="16"/>
 <wire x1="18.8214" y1="18.415" x2="18.6182" y2="18.2118" width="0.2032" layer="16"/>
+<wire x1="18.8776" y1="17.3376" x2="29.1614" y2="13.596" width="0" layer="19" extent="1-1"/>
+<wire x1="11.557" y1="18.1124" x2="18.6182" y2="18.2118" width="0" layer="19" extent="1-1"/>
 </signal>
 <signal name="USB_D+">
