File: PCB/MotionDetectorCamera.sch (EAGLE design)
At the start: 170 parts, among them J1 S-MOUNT-LENS-HOLDER, J2 MINI-USB-JACK, Q1 PMOS-NEXPERIA-SOT1220, Q2 PMOS-NEXPERIA-SOT1220, Q3 PMOS-NEXPERIA-SOT1220, U1 TI-TPS6280XYKAR, U10 TI-TPS22919DCK, U11 TI-TPS22919DCK, U12 STM-STM32F730, U13 MICROCHIP-MIC550X, U14 TI-MSP430FR2422IRHL, U15 TI-SN74AXC4T774RSV, U16 TI-TPS22919DCK, U17 DIODESINC-DT1446-04V-7, U18 TI-SN74LVC1G126, U19 PANASONIC-EKMB110711X, U2 TI-TPS6280XYKAR, U20 TI-TPS22919DCK, U3 TI-TPS63805YFFR, U4 LATTICE-ICE40HX4K-BG121, U5 ON-AR0330CS1C12SPKA0, U6 ALLIANCE-AS4C8M16MSA-6BIN, U7 MAXIM-MAX40203ANS+T, U8 TI-TPS22919DCK, U9 MICROSD-SOCKET, X1 SITIME-SIT8021, X2 SITIME-SIT8021, X3 EPSON-MC-306

Commit message: Cleanup
Parts:
- removed C75: 10u, EagleLibrary:CAPACITOR0805
- removed C76: 100n, EagleLibrary:CAPACITOR0402
- added C83: 2.2u, EagleLibrary:CAPACITOR0402
- added TP11: TEST-POINT, EagleLibrary:TEST-POINT
Connections:
- new net N$22: TP11.X, U14B.P1.1/UCB0CLK/ACLK/A1/VREF+
- net GND: now also C83.2; no longer C75.2, C76.2
- net VDD_A: now also C83.1; no longer C75.1, C76.1
Other:
- note added: "ACLK test point"
- note removed: "Leaving P1.1 unpopulated so ACLK can be observed without side-effects"
Changed lines of the file:
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@@
-<attribute name="PN" value="GRM155R61H104KE19D"/>
-</part>
-<part name="C75" library="EagleLibrary" deviceset="CAPACITOR" device="0805" value="10u">
-<attribute name="MFG" value="KEMET"/>
-<attribute name="PN" value="C0805C106K8PACTU"/>
-</part>
-<part name="C76" library="EagleLibrary" deviceset="CAPACITOR" device="0402" value="100n">
-<attribute name="MFG" value="Murata"/>
 <attribute name="PN" value="GRM155R61H104KE19D"/>
 </part>
@@
 </part>
 <part name="C82" library="EagleLibrary" deviceset="CAPACITOR" device="0402" value="2.2u">
+<attribute name="MFG" value="Taiyo Yuden"/>
+<attribute name="PN" value="TMK105CBJ225KV-F"/>
+</part>
+<part name="TP11" library="EagleLibrary" deviceset="TEST-POINT" device=""/>
+<part name="C83" library="EagleLibrary" deviceset="CAPACITOR" device="0402" value="2.2u">
 <attribute name="MFG" value="Taiyo Yuden"/>
 <attribute name="PN" value="TMK105CBJ225KV-F"/>
@@
 <description>MSP</description>
 <plain>
-<text x="35.052" y="77.724" size="0.762" layer="95" align="top-right">Leaving P1.1 unpopulated so ACLK can
-be observed without side-effects</text>
 <text x="106.426" y="128.524" size="1.016" layer="95" align="top-left">From "MSP430TM 32-kHz Crystal Oscillators",
 section "Effective Load Capacitance":
@@
 capacitance variation due to temperature
 and DC bias</text>
+<text x="0.254" y="76.962" size="0.762" layer="95">ACLK
+test point</text>
 </plain>
 <instances>
@@
 <attribute name="NAME" x="-65.786" y="83.439" size="1.778" layer="95"/>
 <attribute name="VALUE" x="-65.786" y="80.899" size="1.778" layer="96"/>
+</instance>
+<instance part="TP11" gate="G$1" x="5.08" y="76.2" smashed="yes" rot="R90">
+<attribute name="NAME" x="5.08" y="76.2" size="1.778" layer="95" rot="R180"/>
 </instance>
 </instances>
@@
 <wire x1="129.54" y1="66.04" x2="127" y2="66.04" width="0.1524" layer="91"/>
 <label x="127" y="66.04" size="1.778" layer="95" align="bottom-right"/>
+</segment>
+</net>
+<net name="N$22" class="0">
+<segment>
+<pinref part="U14" gate="B" pin="P1.1/UCB0CLK/ACLK/A1/VREF+"/>
+<pinref part="TP11" gate="G$1" pin="X"/>
+<wire x1="35.56" y1="76.2" x2="5.08" y2="76.2" width="0.1524" layer="91"/>
 </segment>
 </net>
@@
 <attribute name="PN" x="0" y="-10.16" size="1.778" layer="95"/>
 </instance>
-<instance part="C75" gate="G$1" x="-27.94" y="-2.54" smashed="yes">
-<attribute name="NAME" x="-25.654" y="-2.667" size="1.778" layer="95"/>
-<attribute name="VALUE" x="-25.654" y="-5.207" size="1.778" layer="96"/>
-<attribute name="MFG" x="-27.94" y="-2.54" size="1.778" layer="96" display="off"/>
-<attribute name="PN" x="-27.94" y="-2.54" size="1.778" layer="96" display="off"/>
-</instance>
-<instance part="C76" gate="G$1" x="-35.56" y="-2.54" smashed="yes">
-<attribute name="PN" x="-5.08" y="0" size="1.778" layer="96" display="off"/>
-<attribute name="NAME" x="-43.688" y="-3.175" size="1.778" layer="95"/>
-<attribute name="VALUE" x="-43.688" y="-5.715" size="1.778" layer="96"/>
-<attribute name="MFG" x="-35.56" y="-2.54" size="1.778" layer="96" display="off"/>
+<instance part="C83" gate="G$1" x="-17.78" y="-2.54" smashed="yes">
+<attribute name="PN" x="-35.56" y="2.54" size="1.778" layer="96" display="off"/>
+<attribute name="NAME" x="-21.082" y="-2.921" size="1.778" layer="95" align="bottom-right"/>
+<attribute name="VALUE" x="-21.082" y="-5.461" size="1.778" layer="96" align="bottom-right"/>
+<attribute name="MFG" x="-35.56" y="2.54" size="1.778" layer="96" display="off"/>
 </instance>
 </instances>
@@
 </segment>
 <segment>
-<pinref part="C75" gate="G$1" pin="1"/>
-<label x="-35.56" y="0" size="1.778" layer="95"/>
-<pinref part="C76" gate="G$1" pin="1"/>
-<wire x1="-27.94" y1="0" x2="-35.56" y2="0" width="0.1524" layer="91"/>
+<pinref part="C83" gate="G$1" pin="1"/>
+<wire x1="-17.78" y1="0" x2="-17.78" y2="2.54" width="0.1524" layer="91"/>
+<label x="-17.78" y="2.54" size="1.778" layer="95" align="bottom-right"/>
 </segment>
 </net>
@@
 </segment>
 <segment>
-<pinref part="C75" gate="G$1" pin="2"/>
-<label x="-35.56" y="-7.62" size="1.778" layer="95" align="top-left"/>
-<pinref part="C76" gate="G$1" pin="2"/>
-<wire x1="-35.56" y1="-7.62" x2="-27.94" y2="-7.62" width="0.1524" layer="91"/>
-</segment>
-</net>
+<pinref part="C83" gate="G$1" pin="2"/>
+<wire x1="-17.78" y1="-7.62" x2="-17.78" y2="-10.16" width="0.1524" layer="91"/>
+<label x="-17.78" y="-10.16" size="1.778" layer="95" align="bottom-right"/>
+</segment>
+</net>

Commit message: Add jumpers to VDD_BAT, VDD_USB, VDD_A, VDD_B, so we can measure current consumption
Parts:
- removed R35, R38: 0, EagleLibrary:RESISTOR0805
- added J3, J4, J5, J6: JUMPER, EagleLibrary:JUMPER
Connections:
- new net N$24: C78.1, J6.2, U20.EN, U20.VIN
- new net VDD_BAT_IN: J5.1
- net N$15: now also J4.1; no longer R38.2
- net N$9: now also J3.1; no longer R35.2
- net VDD_1V9: now also C79.1, C82.1
- net VDD_2V8: now also C80.1, C81.1
- net VDD_A: now also J3.2; no longer R35.1
- net VDD_B: now also J4.2; no longer R38.1
- net VDD_BAT: now also J5.2
- net VDD_USB_IN: now also J6.1; no longer C78.1, C79.1, C80.1, C81.1, C82.1, U20.EN, U20.VIN
Other:
- moved on the sheet: C74, C78, C79, C80, C81, C82, D1, Q1, Q2, Q3, R23, R24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
