File: PCB/MotionDetectorCamera.sch (EAGLE design)
At the start: 184 parts, among them J1 JUMPER-SOLDER, J12 JUMPER-AMPHENOL-10129380-9020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, J13 JUMPER-AMPHENOL-10129380-9020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, J14 JUMPER-AMPHENOL-10129380-9020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, J15 JUMPER-AMPHENOL-10129380-9020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, J2 JUMPER-SOLDER, J4 JUMPER-AMPHENOL-10129380-9020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, J5 JUMPER-SOLDER, J6 S-MOUNT-LENS-HOLDER, J7 MICROSD-SOCKET, J8 MINI-USB-JACK, Q10 PMOS-NEXPERIA-SOT1220, Q2 PMOS-NEXPERIA-SOT1220, Q3 PMOS-NEXPERIA-SOT1220, U1 NEXPERIA-74LVC1G98-BUFFER, U10 TI-TPS22919DCK, U11 TI-TPS2116, U12 TI-MSP430FR2422IRHL, U14 PANASONIC-EKMB110711X, U15 LATTICE-ICE40HX4K-BG121, U16 MICROCHIP-MCP7383X, U17 ON-AR0330CS1C12SPKA0, U18 ALLIANCE-AS4C8M16MSA-6BIN, U19 STM-STM32F730, U2 DIODESINC-AP7350, U20 DIODESINC-DT1446-04V-7, U21 NXP-NTB0102, U22 NXP-NTB0102, U23 TI-TPS6280XYKAR, U24 NEXPERIA-74LVC1G98-OR-INV-INP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, U28 NEXPERIA-74LVC1G98-NOR, U3 TI-TPS6280XYKAR, U30 TI-TPS22919DCK, U4 TI-TPS6280XYKAR, U5 WINBOND-W25Q40EW, U6 TI-TPS22919DCK, U7 TI-TPS22919DCK, U8 TI-TPS22919DCK, U9 TI-TPS22919DCK, X1 EPSON-FC-135, X2 SITIME-SIT8021, X3 SITIME-SIT8021

Commit message: Progress
Connections:
- new net BAT_CHRG_STAT: U16.STAT
Other:
- moved on the sheet: C88, R2, U16
Changed lines of the file:
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@@
 <attribute name="PN" value="GRM155R61H104KE19D"/>
-</part>
-<part name="C88" library="EagleLibrary" deviceset="CAPACITOR" device="0805" value="10u">
-<attribute name="MFG" value="Samsung"/>
-<attribute name="PN" value="CL21A106KOQNNNE"/>
 </part>
 <part name="C91" library="EagleLibrary" deviceset="CAPACITOR" device="0805" value="10u">
@@
 <attribute name="MFG" value="Murata"/>
 <attribute name="PN" value="GRM155R61H104KE19D"/>
+</part>
+<part name="C88" library="EagleLibrary" deviceset="CAPACITOR" device="0805" value="10u">
+<attribute name="MFG" value="Samsung"/>
+<attribute name="PN" value="CL21A106KOQNNNE"/>
 </part>
 </parts>
@@
 <wire x1="231.14" y1="378.46" x2="177.8" y2="378.46" width="0.1524" layer="95"/>
 <text x="180.594" y="336.296" size="2.54" layer="95" align="top-left">Battery reverse polarity protection</text>
-<text x="157.988" y="391.922" size="1.016" layer="95" align="top-left">Resistor sets battery
+<text x="155.448" y="391.922" size="1.016" layer="95" align="top-left">Resistor sets battery
 charge current:
 I = 1000 / R
@@
 <attribute name="PN" x="233.755" y="436.7559" size="1.778" layer="95" ratio="10" rot="SR0"/>
 </instance>
-<instance part="U16" gate="G$1" x="175.26" y="414.02" smashed="yes">
-<attribute name="NAME" x="175.335" y="414.9119" size="1.778" layer="95" ratio="10" rot="SR0"/>
-<attribute name="PN" x="175.335" y="393.5759" size="1.778" layer="95" ratio="10" rot="SR0"/>
-</instance>
-<instance part="R2" gate="G$1" x="162.56" y="401.32" smashed="yes" rot="R90">
-<attribute name="NAME" x="160.528" y="401.32" size="1.778" layer="95" align="top-right"/>
-<attribute name="VALUE" x="160.528" y="398.78" size="1.778" layer="96" align="top-right"/>
+<instance part="U16" gate="G$1" x="172.72" y="414.02" smashed="yes">
+<attribute name="NAME" x="172.795" y="414.9119" size="1.778" layer="95" ratio="10" rot="SR0"/>
+<attribute name="PN" x="172.795" y="393.5759" size="1.778" layer="95" ratio="10" rot="SR0"/>
+</instance>
+<instance part="R2" gate="G$1" x="160.02" y="401.32" smashed="yes" rot="R90">
+<attribute name="NAME" x="157.988" y="401.32" size="1.778" layer="95" align="top-right"/>
+<attribute name="VALUE" x="157.988" y="398.78" size="1.778" layer="96" align="top-right"/>
 </instance>
 <instance part="Q2" gate="G$1" x="220.98" y="358.14" smashed="yes" rot="R90">
@@
 <attribute name="NAME" x="328.168" y="468.376" size="1.778" layer="95" rot="MR0"/>
 </instance>
-<instance part="C88" gate="G$1" x="208.28" y="408.94" smashed="yes">
-<attribute name="NAME" x="211.074" y="408.559" size="1.778" layer="95"/>
-<attribute name="VALUE" x="211.074" y="406.019" size="1.778" layer="96"/>
-<attribute name="MFG" x="208.28" y="408.94" size="1.778" layer="96" display="off"/>
-<attribute name="PN" x="208.28" y="408.94" size="1.778" layer="96" display="off"/>
-</instance>
 <instance part="C91" gate="G$1" x="264.16" y="459.74" smashed="yes">
 <attribute name="NAME" x="266.954" y="459.359" size="1.778" layer="95"/>
@@
 <attribute name="NAME" x="343.662" y="459.359" size="1.778" layer="95" rot="MR0" align="bottom-right"/>
 <attribute name="VALUE" x="343.662" y="456.819" size="1.778" layer="96" rot="MR0" align="bottom-right"/>
+</instance>
+<instance part="C88" gate="G$1" x="205.74" y="421.64" smashed="yes">
+<attribute name="NAME" x="208.534" y="421.259" size="1.778" layer="95"/>
+<attribute name="VALUE" x="208.534" y="418.719" size="1.778" layer="96"/>
+<attribute name="MFG" x="205.74" y="421.64" size="1.778" layer="96" display="off"/>
+<attribute name="PN" x="205.74" y="421.64" size="1.778" layer="96" display="off"/>
 </instance>
 </instances>
@@
 <segment>
 <pinref part="U16" gate="G$1" pin="GND"/>
-<wire x1="172.72" y1="401.32" x2="170.18" y2="401.32" width="0.1524" layer="91"/>
-<label x="170.18" y="401.32" size="1.778" layer="95" align="bottom-right"/>
+<wire x1="170.18" y1="401.32" x2="167.64" y2="401.32" width="0.1524" layer="91"/>
+<label x="167.64" y="401.32" size="1.778" layer="95" align="bottom-right"/>
 </segment>
 <segment>
 <pinref part="R2" gate="G$1" pin="1"/>
-<wire x1="162.56" y1="396.24" x2="162.56" y2="393.7" width="0.1524" layer="91"/>
-<label x="162.56" y="393.7" size="1.778" layer="95"/>
+<wire x1="160.02" y1="396.24" x2="160.02" y2="393.7" width="0.1524" layer="91"/>
+<label x="160.02" y="393.7" size="1.778" layer="95"/>
 </segment>
 <segment>
@@
 </segment>
 <segment>
-<pinref part="C88" gate="G$1" pin="2"/>
-<wire x1="208.28" y1="403.86" x2="208.28" y2="401.32" width="0.1524" layer="91"/>
-<label x="208.28" y="401.32" size="1.778" layer="95"/>
-</segment>
-<segment>
 <wire x1="223.52" y1="467.36" x2="223.52" y2="464.82" width="0.1524" layer="91"/>
 <label x="223.52" y="464.82" size="1.778" layer="95"/>
@@
 <wire x1="340.36" y1="454.66" x2="340.36" y2="452.12" width="0.1524" layer="91"/>
 <label x="340.36" y="452.12" size="1.778" layer="95" rot="MR0" align="bottom-right"/>
+</segment>
+<segment>
+<pinref part="C88" gate="G$1" pin="2"/>
+<wire x1="205.74" y1="416.56" x2="205.74" y2="414.02" width="0.1524" layer="91"/>
+<label x="205.74" y="414.02" size="1.778" layer="95"/>
 </segment>
 </net>
@@
 <segment>
 <pinref part="U16" gate="G$1" pin="VDD"/>
-<wire x1="172.72" y1="411.48" x2="149.86" y2="411.48" width="0.1524" layer="91"/>
+<wire x1="170.18" y1="411.48" x2="149.86" y2="411.48" width="0.1524" layer="91"/>
 <wire x1="149.86" y1="411.48" x2="149.86" y2="452.12" width="0.1524" layer="91"/>
 <pinref part="R5" gate="G$1" pin="1"/>
@@
 <junction x="195.58" y="373.38"/>
 <pinref part="U16" gate="G$1" pin="VBAT"/>
-<wire x1="198.12" y1="411.48" x2="208.28" y2="411.48" width="0.1524" layer="91"/>
-<wire x1="208.28" y1="411.48" x2="220.98" y2="411.48" width="0.1524" layer="91"/>
+<wire x1="195.58" y1="411.48" x2="220.98" y2="411.48" width="0.1524" layer="91"/>
 <wire x1="220.98" y1="411.48" x2="220.98" y2="373.38" width="0.1524" layer="91"/>
 <junction x="220.98" y="373.38"/>
@@
 <pinref part="U11" gate="G$1" pin="VIN2"/>
 <wire x1="220.98" y1="447.04" x2="231.14" y2="447.04" width="0.1524" layer="91"/>
+</segment>
+<segment>
 <pinref part="C88" gate="G$1" pin="1"/>
-<junction x="208.28" y="411.48"/>
+<wire x1="205.74" y1="424.18" x2="205.74" y2="426.72" width="0.1524" layer="91"/>
+<label x="205.74" y="426.72" size="1.778" layer="95" align="top-left"/>
 </segment>
 </net>
@@
 <pinref part="R2" gate="G$1" pin="2"/>
 <pinref part="U16" gate="G$1" pin="PROG"/>
-<wire x1="162.56" y1="406.4" x2="172.72" y2="406.4" width="0.1524" layer="91"/>
+<wire x1="160.02" y1="406.4" x2="170.18" y2="406.4" width="0.1524" layer="91"/>
 </segment>
 </net>
@@
 </segment>
 </net>
+<net name="BAT_CHRG_STAT" class="0">
+<segment>
+<pinref part="U16" gate="G$1" pin="STAT"/>
+<wire x1="195.58" y1="406.4" x2="198.12" y2="406.4" width="0.1524" layer="91"/>
+<label x="198.12" y="406.4" size="1.778" layer="95"/>
+</segment>
+</net>

Commit message: Progress
Parts:
- added Q1: PMOS-NEXPERIA-SOT1220, EagleLibrary:PMOS-NEXPERIA-SOT1220
- added R35: 100k, EagleLibrary:RESISTOR0402
- R5, R6: value 100k -> 300k; MFG Stackpole -> (none); PN RMCF0402JT100K -> (none)
Connections:
- removed net N$36: R5.2, R6.1
- removed net N$39: R6.2, R7.1
- new net BAT_CHRG_LVL: R35.1, R6.2
- new net BAT_CHRG_LVL_EN_: Q1.G, R7.2
- new net N$46: Q1.D, R6.1
- net GND: now also R35.2
- net N$42: now also R5.2; no longer R7.2
- net VDD_BAT: now also Q1.S, R7.1
Other:
- note added: "Battery Charge Level"
- note added: "The MOSFET prevents the battery drain caused by the voltage divider until the time comes that we actually need to measure the battery voltage. When we actually want to sample BAT_CHRG_LVL and accept the ensuing battery drain, STM32 asserts BAT_CHRG_LVL_EN_. STM32 is only running when we're connected to USB and therefore charging the battery, in which case we're not concerned with the small amount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"
- moved on the sheet: J4, Q2, Q3, R3, R4, R5, R6, R7, R8
