File: PCB/MotionDetectorCamera.sch (EAGLE design)
At the start: 186 parts, among them J1 JUMPER-SOLDER, J10 MICROSD-SOCKET, J11 USB-C-JACK, J2 JUMPER-SOLDER, J3 JUMPER-SOLDER, J4 JUMPER-SOLDER, J5 JST-SM02B-SRSS-TB, J6 JUMPER-SOLDER, J7 JUMPER-SOLDER, J8 JUMPER-SOLDER, J9 S-MOUNT-LENS-HOLDERM12LENSES-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, Q1 PMOS-NEXPERIA-SOT1220, Q2 PMOS-NEXPERIA-SOT1220, Q3 PMOS-NEXPERIA-SOT1220, U1 TI-TPS2116, U10 TI-TPS22919DCK, U11 TI-TPS62A01, U13 TI-TPS22919DCK, U14 TI-TPS22919DCK, U15 TI-MSP430FR2422IRHL, U16 NXP-NTB0102, U17 NXP-NTB0102, U18 PANASONIC-EKMB110711X, U19 LATTICE-ICE40HX4K-BG121, U2 DIODESINC-AP7350, U20 WINBOND-W25Q40EW, U21 NEXPERIA-74LVC1G98-OR-INV-INP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, U22 NEXPERIA-74LVC1G98-BUFFER, U23 ON-AR0330CS1C12SPKA0, U24 ALLIANCE-AS4C8M16MSA-6BIN, U25 STM-STM32F730, U26 DIODESINC-DT1446-04V-7, U27 NEXPERIA-74LVC1G98-BUFFER, U3 NEXPERIA-74LVC1G98-NOR, U4 MICROCHIP-MCP7383X, U5 EATON-STN101, U6 TI-TPS62A01, U7 TI-TPS62A01, U9 TI-TPS22919DCK, X1 EPSON-FC-135, X2 SITIME-SIT8021, X3 SITIME-SIT8021

Commit message: Layout progress
Connections:
- removed net MSP_RUN: U15C.PA.D/P2.5/UCB0SIMO/UCB0SDA/A7, U25H.PH1_H1
- new net MSP_HOST_MODE_: U15B.PA.0/P1.0/UCB0STE/A0/VEREF+, U25E.PE5_B2
- net ICE_MSP_SPI_CLK_X: now also U15C.PA.C/P2.4/TA1CLK/UCB0CLK/A6; no longer U15B.PA.6/P1.6/UCA0CLK/TA0CLK/TDI/TCLK
- net ICE_MSP_SPI_DATA_X: now also U15C.PA.D/P2.5/UCB0SIMO/UCB0SDA/A7, U15C.PA.E/P2.6/UCB0SOMI/UCB0SCL; no longer U15B.PA.4/P1.4/UCA0TXD/UCA0SIMO/TA0.1/TCK, U15B.PA.5/P1.5/UCA0RXD/UCA0SOMI/TA0.2/TMS
- net VDD_B_1V8_IMG_SD_EN: now also U15B.PA.6/P1.6/UCA0CLK/TA0CLK/TDI/TCLK; no longer U15B.PA.0/P1.0/UCB0STE/A0/VEREF+
- net VDD_B_2V8_IMG_SD_EN: now also U15B.PA.5/P1.5/UCA0RXD/UCA0SOMI/TA0.2/TMS; no longer U15B.PA.2/P1.2/UCB0SIMO/UCB0SDA/SMCLK/A2/VEREF-
- net VDD_B_EN: now also U15B.PA.4/P1.4/UCA0TXD/UCA0SIMO/TA0.1/TCK; no longer U15B.PA.1/P1.1/UCB0CLK/ACLK/A1/VREF+
Changed lines of the file:
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@@
 <net name="ICE_MSP_SPI_DATA_X" class="0">
 <segment>
-<pinref part="U15" gate="B" pin="PA.4/P1.4/UCA0TXD/UCA0SIMO/TA0.1/TCK"/>
-<pinref part="U15" gate="B" pin="PA.5/P1.5/UCA0RXD/UCA0SOMI/TA0.2/TMS"/>
-<wire x1="35.56" y1="68.58" x2="35.56" y2="66.04" width="0.1524" layer="91"/>
-<wire x1="35.56" y1="66.04" x2="33.02" y2="66.04" width="0.1524" layer="91"/>
-<junction x="35.56" y="66.04"/>
-<label x="33.02" y="66.04" size="1.778" layer="95" align="bottom-right"/>
-</segment>
-<segment>
 <wire x1="101.6" y1="0" x2="99.06" y2="0" width="0.1524" layer="91"/>
 <label x="99.06" y="0" size="1.778" layer="95" align="bottom-right"/>
 <pinref part="U17" gate="G$1" pin="B1"/>
 </segment>
-</net>
-<net name="ICE_MSP_SPI_CLK_X" class="0">
 <segment>
-<pinref part="U15" gate="B" pin="PA.6/P1.6/UCA0CLK/TA0CLK/TDI/TCLK"/>
-<wire x1="35.56" y1="63.5" x2="33.02" y2="63.5" width="0.1524" layer="91"/>
-<label x="33.02" y="63.5" size="1.778" layer="95" align="bottom-right"/>
+<wire x1="129.54" y1="66.04" x2="129.54" y2="63.5" width="0.1524" layer="91"/>
+<wire x1="129.54" y1="63.5" x2="127" y2="63.5" width="0.1524" layer="91"/>
+<junction x="129.54" y="63.5"/>
+<label x="127" y="63.5" size="1.778" layer="95" align="bottom-right"/>
+<pinref part="U15" gate="C" pin="PA.D/P2.5/UCB0SIMO/UCB0SDA/A7"/>
+<pinref part="U15" gate="C" pin="PA.E/P2.6/UCB0SOMI/UCB0SCL"/>
 </segment>
+</net>
+<net name="ICE_MSP_SPI_CLK_X" class="0">
 <segment>
 <wire x1="101.6" y1="-5.08" x2="99.06" y2="-5.08" width="0.1524" layer="91"/>
@@
 <pinref part="U17" gate="G$1" pin="B2"/>
 </segment>
+<segment>
+<wire x1="129.54" y1="68.58" x2="127" y2="68.58" width="0.1524" layer="91"/>
+<label x="127" y="68.58" size="1.778" layer="95" align="bottom-right"/>
+<pinref part="U15" gate="C" pin="PA.C/P2.4/TA1CLK/UCB0CLK/A6"/>
+</segment>
 </net>
 <net name="VDD_B_1V8" class="0">
@@
 </segment>
 </net>
-<net name="VDD_B_1V8_IMG_SD_EN" class="0">
-<segment>
-<wire x1="35.56" y1="78.74" x2="33.02" y2="78.74" width="0.1524" layer="91"/>
-<label x="33.02" y="78.74" size="1.778" layer="95" align="bottom-right"/>
-<pinref part="U15" gate="B" pin="PA.0/P1.0/UCB0STE/A0/VEREF+"/>
-</segment>
-</net>
-<net name="VDD_B_2V8_IMG_SD_EN" class="0">
-<segment>
-<pinref part="U15" gate="B" pin="PA.2/P1.2/UCB0SIMO/UCB0SDA/SMCLK/A2/VEREF-"/>
-<wire x1="35.56" y1="73.66" x2="33.02" y2="73.66" width="0.1524" layer="91"/>
-<label x="33.02" y="73.66" size="1.778" layer="95" align="bottom-right"/>
-</segment>
-</net>
 <net name="N$14" class="0">
 <segment>
@@
 </segment>
 </net>
-<net name="VDD_B_EN" class="0">
-<segment>
-<wire x1="35.56" y1="76.2" x2="33.02" y2="76.2" width="0.1524" layer="91"/>
-<label x="33.02" y="76.2" size="1.778" layer="95" align="bottom-right"/>
-<pinref part="U15" gate="B" pin="PA.1/P1.1/UCB0CLK/ACLK/A1/VREF+"/>
-</segment>
-</net>
-<net name="MSP_RUN" class="0">
-<segment>
-<pinref part="U15" gate="C" pin="PA.D/P2.5/UCB0SIMO/UCB0SDA/A7"/>
-<wire x1="129.54" y1="66.04" x2="127" y2="66.04" width="0.1524" layer="91"/>
-<label x="127" y="66.04" size="1.778" layer="95" align="bottom-right"/>
-</segment>
-</net>
 <net name="MSP_SBW_EN" class="0">
 <segment>
@@
 </segment>
 </net>
+<net name="VDD_B_EN" class="0">
+<segment>
+<wire x1="35.56" y1="68.58" x2="33.02" y2="68.58" width="0.1524" layer="91"/>
+<label x="33.02" y="68.58" size="1.778" layer="95" align="bottom-right"/>
+<pinref part="U15" gate="B" pin="PA.4/P1.4/UCA0TXD/UCA0SIMO/TA0.1/TCK"/>
+</segment>
+</net>
+<net name="VDD_B_2V8_IMG_SD_EN" class="0">
+<segment>
+<wire x1="35.56" y1="66.04" x2="33.02" y2="66.04" width="0.1524" layer="91"/>
+<label x="33.02" y="66.04" size="1.778" layer="95" align="bottom-right"/>
+<pinref part="U15" gate="B" pin="PA.5/P1.5/UCA0RXD/UCA0SOMI/TA0.2/TMS"/>
+</segment>
+</net>
+<net name="VDD_B_1V8_IMG_SD_EN" class="0">
+<segment>
+<wire x1="35.56" y1="63.5" x2="33.02" y2="63.5" width="0.1524" layer="91"/>
+<label x="33.02" y="63.5" size="1.778" layer="95" align="bottom-right"/>
+<pinref part="U15" gate="B" pin="PA.6/P1.6/UCA0CLK/TA0CLK/TDI/TCLK"/>
+</segment>
+</net>
+<net name="MSP_HOST_MODE_" class="0">
+<segment>
+<wire x1="35.56" y1="78.74" x2="33.02" y2="78.74" width="0.1524" layer="91"/>
+<label x="33.02" y="78.74" size="1.778" layer="95" align="bottom-right"/>
+<pinref part="U15" gate="B" pin="PA.0/P1.0/UCB0STE/A0/VEREF+"/>
+</segment>
+</net>
 </nets>
 </sheet>
@@
 </segment>
 </net>
-<net name="MSP_RUN" class="0">
-<segment>
-<pinref part="U25" gate="H" pin="PH1_H1"/>
-<wire x1="170.18" y1="-76.2" x2="172.72" y2="-76.2" width="0.1524" layer="91"/>
-<label x="172.72" y="-76.2" size="1.778" layer="95"/>
-</segment>
-</net>
 <net name="MSP_SBW_EN" class="0">
 <segment>
@@
 </segment>
 </net>
+<net name="MSP_HOST_MODE_" class="0">
+<segment>
+<wire x1="2.54" y1="-86.36" x2="5.08" y2="-86.36" width="0.1524" layer="91"/>
+<label x="5.08" y="-86.36" size="1.778" layer="95"/>
+<pinref part="U25" gate="E" pin="PE5_B2"/>
+</segment>
+</net>

Commit message: Layout progress
Parts:
- J5: MFG HX (Zhejiang Yueqing Hongxing Elec) -> (none); MFG2 HDGC -> (none); PN HX20007-2AWB -> (none); PN2 HDGC2001WR-S-2P -> (none)
Changed lines of the file:
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@@
 <attribute name="PN" value="STN101050B101"/>
 </part>
-<part name="J5" library="EagleLibrary" deviceset="JST-SM02B-SRSS-TB" device="">
-<attribute name="MFG" value="HX (Zhejiang Yueqing Hongxing Elec)"/>
-<attribute name="MFG2" value="HDGC"/>
-<attribute name="PN" value="HX20007-2AWB"/>
-<attribute name="PN2" value="HDGC2001WR-S-2P"/>
-</part>
+<part name="J5" library="EagleLibrary" deviceset="JST-SM02B-SRSS-TB" device=""/>
 <part name="J11" library="EagleLibrary" deviceset="USB-C-JACK" device=""/>
 <part name="R33" library="EagleLibrary" deviceset="RESISTOR" device="0402" value="5.1k">
@@
 </instance>
 <instance part="J5" gate="G$1" x="124.46" y="355.6" smashed="yes">
-<attribute name="MFG" x="124.46" y="355.6" size="1.778" layer="96" display="off"/>
-<attribute name="MFG2" x="124.46" y="355.6" size="1.778" layer="96" display="off"/>
-<attribute name="PN2" x="124.46" y="355.6" size="1.778" layer="96" display="off"/>
 <attribute name="PN" x="124.46" y="337.82" size="1.778" layer="95"/>
 <attribute name="NAME" x="124.46" y="358.14" size="1.778" layer="95" align="top-left"/>

Commit message: Layout progress
Parts:
- removed C38: 100n, EagleLibrary:CAPACITOR0402
Connections:
- net GND: no longer C38.2
- net VDD_B_1V8: no longer C38.1
Other:
- moved on the sheet: C32, C33, C34, C35, C39, C40, C41
