File: PCB/MotionDetectorCamera-Rev4.sch (EAGLE design)
At the start: 189 parts, among them J1 JUMPER-SOLDER, J12 JUMPER-SOLDER, J13 JUMPER-SOLDER, J14 JUMPER-AMPHENOL-10129380-9020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, J15 JUMPER-SOLDER, J2 JUMPER-SOLDER, J3 JST-PH-2, J4 USB-C-JACK, J5 JUMPER-SOLDER, J6 S-MOUNT-LENS-HOLDER, J7 MICROSD-SOCKET, Q1 PMOS-NEXPERIA-SOT1220, Q10 PMOS-NEXPERIA-SOT1220, Q2 PMOS-NEXPERIA-SOT1220, Q3 PMOS-NEXPERIA-SOT1220, U1 NEXPERIA-74LVC1G98-BUFFER, U10 TI-TPS22919DCK, U11 TI-TPS2116, U12 TI-MSP430FR2422IRHL, U13 EATON-STN101, U14 PANASONIC-EKMB110711X, U15 LATTICE-ICE40HX4K-BG121, U16 MICROCHIP-MCP7383X, U17 ON-AR0330CS1C12SPKA0, U18 ALLIANCE-AS4C8M16MSA-6BIN, U19 STM-STM32F730, U2 DIODESINC-AP7350, U20 DIODESINC-DT1446-04V-7, U21 NXP-NTB0102, U22 NXP-NTB0102, U23 TI-TPS6280XYKAR, U24 NEXPERIA-74LVC1G98-OR-INV-INP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, U28 NEXPERIA-74LVC1G98-NOR, U3 TI-TPS6280XYKAR, U30 TI-TPS22919DCK, U4 TI-TPS6280XYKAR, U5 WINBOND-W25Q40EW, U6 TI-TPS22919DCK, U7 TI-TPS22919DCK, U8 TI-TPS22919DCK, U9 TI-TPS22919DCK, X1 EPSON-FC-135, X2 SITIME-SIT8021, X3 SITIME-SIT8021

Commit message: Layout progress
Parts:
- removed C89, C90: 2.2u, EagleLibrary:CAPACITOR0402
- removed C91: 10u, EagleLibrary:CAPACITOR0805
- removed C92, C93: 100n, EagleLibrary:CAPACITOR0402
- removed J12, J13, J15: JUMPER-SOLDER, EagleLibrary:JUMPER-SOLDER
- removed J14: JUMPER-AMPHENOL-10129380-902002ALF, EagleLibrary:JUMPER-AMPHENOL-10129380-902002ALF
- removed L4: 470n, EagleLibrary:INDUCTOR0806
- removed Q10: PMOS-NEXPERIA-SOT1220, EagleLibrary:PMOS-NEXPERIA-SOT1220
- removed R33: 86.6k, EagleLibrary:RESISTOR0402
- removed R35, R36: 100k, EagleLibrary:RESISTOR0402
- removed U21, U22: NXP-NTB0102, EagleLibrary:NXP-NTB0102
- removed U23: TI-TPS6280XYKAR, EagleLibrary:TI-TPS6280XYKAR
- removed U24: NEXPERIA-74LVC1G98-OR-INV-INPUT, EagleLibrary:NEXPERIA-74LVC1G98-OR-INV-INPUT
- removed U28: NEXPERIA-74LVC1G98-NOR, EagleLibrary:NEXPERIA-74LVC1G98-NOR
- removed U30: TI-TPS22919DCK, EagleLibrary:TI-TPS22919DCK
- added J8: MINI-USB-JACK, EagleLibrary:MINI-USB-JACK
- added L3: 470n, EagleLibrary:INDUCTOR0806
- C1: value 2.2u -> 10u; device EagleLibrary:CAPACITOR0402 -> EagleLibrary:CAPACITOR0805; MFG Taiyo Yuden -> Samsung; PN TMK105CBJ225KV-F -> CL21A106KOQNNNE
- C11, C12, C13, C14: value 100n -> 10u; device EagleLibrary:CAPACITOR0402 -> EagleLibrary:CAPACITOR0805; MFG Murata -> Samsung; PN GRM155R61H104KE19D -> CL21A106KOQNNNE
- C22, C23: value 22p -> 9p; MFG (none) -> Yageo; PN (none) -> CC0402BRNPO9BN9R0
- C26: value 22p -> 1n; MFG (none) -> Yageo; PN (none) -> CC0402MRX7R9BB102
- C27: value 10u -> 100n; device EagleLibrary:CAPACITOR0805 -> EagleLibrary:CAPACITOR0402; MFG Samsung -> Murata; PN CL21A106KOQNNNE -> GRM155R61H104KE19D
- C88: value 10u -> 4.7u; device EagleLibrary:CAPACITOR0805 -> EagleLibrary:CAPACITOR0603; MFG Samsung -> Taiyo Yuden; PN CL21A106KOQNNNE -> LMK107BJ475KA-T
- D1: value ROHM-RB168MM-40 -> ROHM-RB168MM-40TFTR; device EagleLibrary:ROHM-RB168MM-40 -> EagleLibrary:ROHM-RB168MM-40TFTR
- J1, J2, J5: value JUMPER-SOLDER -> JUMPER; device EagleLibrary:JUMPER-SOLDER -> EagleLibrary:JUMPER
- J3: value JST-PH-2 -> JUMPER; device EagleLibrary:JST-PH-2 -> EagleLibrary:JUMPER; MFG HX (Zhejiang Yueqing Hongxing Elec) -> (none); MFG2 HDGC -> (none); PN HX20007-2AWB -> (none); PN2 HDGC2001WR-S-2P -> (none)
- J4: value USB-C-JACK -> JUMPER; device EagleLibrary:USB-C-JACK -> EagleLibrary:JUMPER
- R1: value 10k -> 3k; PN RC0402JR-0710KL -> AC0402FR-073KL
- R10: value 5.1k -> 91k; MFG (none) -> Bourns; PN (none) -> CR0402-FX-9102GLF
- R11: value 100 -> 47k; MFG Stackpole -> Walsin; PN RMCF0402JT100R -> WR04X473 JTL
- R16, R17: MFG Stackpole -> Bourns; PN RMCF0402JT100R -> CR0402AJW-101GAS
- R2: value 2.7k -> 100k; MFG (none) -> Yageo; PN (none) -> RC0402FR-10100KL
- R3: MFG Stackpole -> Yageo; PN RMCF0402JT100K -> RC0402FR-10100KL
- R4: value 100k -> 3k; MFG Stackpole -> Yageo; PN RMCF0402JT100K -> AC0402FR-073KL
- R5, R6: value 300k -> 0; device EagleLibrary:RESISTOR0402 -> EagleLibrary:RESISTOR0805; MFG (none) -> Yageo; PN (none) -> RC0805JR-070RL
- R7: value 100k -> 12.1k; MFG Stackpole -> Walsin; PN RMCF0402JT100K -> WR04X1212FTL
- R8: value 100k -> 0; device EagleLibrary:RESISTOR0402 -> EagleLibrary:RESISTOR0805; MFG Stackpole -> Yageo; PN RMCF0402JT100K -> RC0805JR-070RL
- R9: value 5.1k -> 422k; MFG (none) -> Bourns; PN (none) -> CR0402-FX-4223GLF
- U1: value NEXPERIA-74LVC1G98-BUFFER -> MAXIM-MAX40203ANS+T; device EagleLibrary:NEXPERIA-74LVC1G98-BUFFER -> EagleLibrary:MAXIM-MAX40203ANS+T; PN 74LVC1G98GW,125 -> (none)
- U11: value TI-TPS2116 -> MICROCHIP-MIC550X; device EagleLibrary:TI-TPS2116 -> EagleLibrary:MICROCHIP-MIC550X; PN TPS2116DRLR -> MIC5504-3.3YM5-TR
- U13: value EATON-STN101 -> TI-SN74AXC4T774RSV; device EagleLibrary:EATON-STN101 -> EagleLibrary:TI-SN74AXC4T774RSV; PN STN101050B101 -> (none)
- U16: value MICROCHIP-MCP7383X -> TI-SN74LVC1G126; device EagleLibrary:MICROCHIP-MCP7383X -> EagleLibrary:TI-SN74LVC1G126; PN MCP73831T-2ACI/OT -> SN74LVC1G126DCKR
- U2: value DIODESINC-AP7350 -> TI-TPS22919DCK; device EagleLibrary:DIODESINC-AP7350 -> EagleLibrary:TI-TPS22919DCK; PN AP7350-33CF4-7 -> (none)
- U5: value WINBOND-W25Q40EW -> TI-TPS63805YFFR; device EagleLibrary:WINBOND-W25Q40EW -> EagleLibrary:TI-TPS63805YFFR; PN W25Q40EWUXIE -> (none)
- X1: value EPSON-FC-135 -> EPSON-MC-306; device EagleLibrary:EPSON-FC-135 -> EagleLibrary:EPSON-MC-306; PN Q13FC13500005 -> MC-306 32.7680K-E3:ROHS
Connections:
- net VDD_B_1V8_IMG_EN renamed VDD_1V9_IMG_EN
- net VDD_B_1V8_SD renamed VDD_1V9_SD
- net VDD_B_2V8_IMG renamed VDD_2V8_IMG
- net VDD_B_2V8_IMG_EN renamed VDD_2V8_IMG_EN
- net VDD_B_2V8_SD renamed VDD_2V8_SD
- net VDD_B_SD_EN renamed VDD_SD_EN
- removed net BAT_CHRG_LVL: R35.1, R6.2, U19C.PC5_P5
- removed net BAT_CHRG_LVL_EN_: Q1.G, R7.2, U19C.PC4_N5
- removed net BAT_CHRG_STAT: U16.STAT, U19C.PC3_M5
- removed net ICE_ST_FLASH_EN: R1.1, U19B.PB7_B5, U24.IN1
- removed net ICE_ST_SPI_D_READY: U15C.L5, U19A.PA7_R3
- removed net MSP_RST_X_: U19B.PB0_R5, U22.A2
- removed net MSP_TEST_X: U19B.PB1_R4, U22.A1
- removed net N$3: C92.1, D1.A, J15.1, U2.VOUT
- removed net N$32: Q2.D, Q3.G, R3.1
- removed net N$33: R11.1, U28.OUT
- removed net N$34: Q10.G, R11.2
- removed net N$35: J4.CC1, R9.1
- removed net N$36: J4.CC2, R10.1
- removed net N$37: C3.1, J5.1, L4.2, U23.VOS
- removed net N$38: R33.2, U23.MODE
- removed net N$40: U24.OUT, U5.CS_
- removed net N$42: R5.2, R8.1, U11.PR1
- removed net N$43: J12.1, Q10.D
- removed net N$46: Q1.D, R6.1
- removed net VDD_A_3V3: C11.1, C12.1, C20.1, C24.1, C25.1, C29.1, J15.2, U12A.VDD, U14.VDD, U21.VCCB, U22.VCCB, U28.VDD, U30.VIN
- removed net VDD_BAT: C88.1, Q1.S, Q2.S, Q3.S, R4.2, R7.1, U11.VIN2, U16.VBAT
- removed net VDD_B_1V2: C30.1, C31.1, C32.1, C33.1, J1.2, R16.2, R17.2, U15E.VCC_D4, U15E.VCC_D8, U15E.VCC_H4, U15E.VCC_H8
- removed net VDD_B_1V8: C14.1, C15.1, C18.1, C19.1, C28.1, C34.1, C35.1, C36.1, C37.1, C38.1, C39.1, C44.1, C61.1, C62.1, C63.1, C64.1, J2.2, R1.2, R18.1, R19.1, U10.VIN, U15E.VCCIO_0_D6, U15E.VCCIO_1_F8, U15E.VCCIO_2_H6, U15E.VCCIO_3_E4, U15E.VCCIO_3_G4, U15E.VCC_SPI_L11, U18A.VDDQ_A7, U18A.VDDQ_B3, U18A.VDDQ_C7, U18A.VDDQ_D3, U18A.VDD_A9, U18A.VDD_E7, U18A.VDD_J9, U21.OE, U21.VCCA, U24.VDD, U5.VCC, U6.VIN, U9.VIN, X2.VDD
- removed net VDD_B_1V8_IMG: C47.1, C52.1, C53.1, C54.1, C55.1, C56.1, C57.1, C58.1, R20.2, R21.1, U1.VDD, U17A.VDD, U17A.VDD_IO, U6.QOD, U6.VOUT
- removed net VDD_B_1V8_STM: C1.1, C13.1, C21.1, C4.1, C67.1, C70.1, C71.1, C72.1, C73.1, C74.1, C75.1, C76.1, C77.1, C80.1, C81.1, C82.1, C83.1, C84.1, C85.1, U10.QOD, U10.VOUT, U19J.PDR_ON_C6, U19K.VBAT_C1, U19K.VDDA_R1, U19K.VDDSDMMC_C8, U19K.VDD_C5, U19K.VDD_C7, U19K.VDD_C9, U19K.VDD_F3, U19K.VDD_G13, U19K.VDD_G3, U19K.VDD_J12, U19K.VDD_J13, U19K.VDD_K4, U19K.VDD_N10, U19K.VDD_N8, U19K.VDD_N9, U19K.VREF+_P1, U22.OE, U22.VCCA, U30.EN, X3.VDD
- removed net VDD_B_2V8: C16.1, C17.1, C40.1, C41.1, J5.2, U15E.VPP_2V5_C10, U7.VIN, U8.VIN
- removed net VDD_B_3V3_STM: C78.1, C79.1, U19K.VDDUSB_H13, U30.QOD, U30.VOUT
- removed net VDD_B_EN: U12C.PA.C/P2.4/TA1CLK/UCB0CLK/A6, U28.IN2
- new net ICE_MSP_SPI_AUX: U13.B3, U15C.K3
- new net ICE_MSP_SPI_AUX_DIR: U12C.PA.A/P2.2/TA1.1/A4, U13.DIR3
- new net ICE_MSP_SPI_AUX_X: U12B.PA.7/P1.7/UCA0STE/TDO, U13.A3
- new net ICE_MSP_SPI_DATA_DIR: U12B.PA.3/P1.3/UCB0SOMI/UCB0SCL/MCLK/A3, U13.DIR1
- new net N$1: J2.2, Q2.D
- new net N$11: R10.2, R9.1, U5.FB
- new net N$12: L3.1, U5.L1
- new net N$13: L3.2, U5.L2
- new net N$15: C3.1, D1.C, J3.1, Q3.D
- new net N$18: C13.1, C14.1, R8.2, R9.2, U5.VOUT
- new net N$19: C2.1, Q1.S, Q2.S, Q3.S, R3.1
- new net N$24: C4.1, J4.2, U2.EN, U2.VIN
- new net N$9: C1.1, J1.1, Q1.D, U1.VOUT
- new net VDD_1V2: C30.1, C31.1, C32.1, C33.1, R16.2, R17.2, R5.1, U15E.VCC_D4, U15E.VCC_D8, U15E.VCC_H4, U15E.VCC_H8
- new net VDD_1V9: C15.1, C18.1, C19.1, C28.1, C34.1, C35.1, C36.1, C37.1, C38.1, C39.1, C44.1, C61.1, C62.1, C63.1, C64.1, R18.1, R19.1, R6.1, U1.EN, U1.VIN, U10.VIN, U13.VCCB, U15E.VCCIO_0_D6, U15E.VCCIO_1_F8, U15E.VCCIO_2_H6, U15E.VCCIO_3_E4, U15E.VCCIO_3_G4, U15E.VCC_SPI_L11, U18A.VDDQ_A7, U18A.VDDQ_B3, U18A.VDDQ_C7, U18A.VDDQ_D3, U18A.VDD_A9, U18A.VDD_E7, U18A.VDD_J9, U6.VIN, U9.VIN, X2.VDD
- new net VDD_1V9_IMG: C47.1, C52.1, C53.1, C54.1, C55.1, C56.1, C57.1, C58.1, R20.2, R21.1, U16.EN, U16.VDD, U17A.VDD, U17A.VDD_IO, U6.QOD, U6.VOUT
- new net VDD_1V9_STM: C67.1, C70.1, C71.1, C72.1, C73.1, C74.1, C75.1, C76.1, C77.1, C80.1, C81.1, C82.1, C83.1, C84.1, C85.1, C88.1, U10.QOD, U10.VOUT, U11.EN, U19J.PDR_ON_C6, U19K.VBAT_C1, U19K.VDDA_R1, U19K.VDDSDMMC_C8, U19K.VDD_C5, U19K.VDD_C7, U19K.VDD_C9, U19K.VDD_F3, U19K.VDD_G13, U19K.VDD_G3, U19K.VDD_J12, U19K.VDD_J13, U19K.VDD_K4, U19K.VDD_N10, U19K.VDD_N8, U19K.VDD_N9, U19K.VREF+_P1, X3.VDD
- new net VDD_2V8: C16.1, C17.1, C40.1, C41.1, R8.1, U15E.VPP_2V5_C10, U7.VIN, U8.VIN
- new net VDD_3V3_STM: C21.1, C78.1, C79.1, U11.VOUT, U19K.VDDUSB_H13
- new net VDD_B_EN_: R4.2, U12C.PA.C/P2.4/TA1CLK/UCB0CLK/A6
- new net VDD_SRC_USB: Q1.G, Q2.G, R1.1, R2.2
- net GND: now also J5.1, J5.2, J8.GND, R10.1, R7.1, U13.EN_, U13.GND, U5.AGND, U5.MODE; no longer C89.2, C90.2, C91.2, C92.2, C93.2, J14.1, J14.2, J3.GND, J3.R, J4.GND, R10.2, R3.2, R33.1, R35.2, R36.2, R8.2, R9.2, U13.2, U21.GND, U22.GND, U23.GND, U24.GND, U28.GND, U30.GND, U4.MODE
- net ICE_IMG_CLK16MHZ: now also U16.IN; no longer U1.IN
- net ICE_MSP_SPI_CLK: now also U13.B2; no longer U21.A1
- net ICE_MSP_SPI_CLK_X: now also U13.A2; no longer U21.B1
- net ICE_MSP_SPI_DATA: now also U13.B1, U15D.K1; no longer U15C.K3, U21.A2
- net ICE_MSP_SPI_DATA_X: now also U13.A1; no longer U21.B2
- net ICE_ST_SPI_CLK: no longer U5.CLK
- net ICE_ST_SPI_CS_: no longer U24.IN2
- net ICE_ST_SPI_D0: no longer U5.DI
- net ICE_ST_SPI_D1: no longer U5.DO
- net IMG_CLK16MHZ: now also U16.OUT; no longer U1.OUT
- net MSP_RST_: now also R11.1, U19B.PB0_R5; no longer U22.B2
- net MSP_TEST: now also U19B.PB1_R4; no longer U22.B1
- net N$16: now also R5.2; no longer J1.1
- net N$21: now also R7.2, U4.MODE; no longer R2.2, U16.PROG
- net N$54: now also J8.VCC; no longer J4.VBUS
- net N$6: now also Q3.G, R3.2, R4.1; no longer L4.1, U23.SW
- net N$8: now also R6.2; no longer J2.1
- net USB_D+: now also J8.D+; no longer J4.D+
- net USB_D-: now also J8.D-; no longer J4.D-
- net VDD_A: now also C24.1, C25.1, C27.1, C29.1, J1.2, R11.2, U12A.VDD, U13.DIR2, U13.VCCA, U14.VDD; no longer C91.1, C93.1, D1.C, Q10.S, U11.VOUT, U2.EN, U2.VIN
- net VDD_B: now also C11.1, C12.1, J3.2, U5.EN, U5.VIN; no longer C2.1, C27.1, J12.2, U23.EN, U23.VIN
- net VDD_BAT_IN: now also J2.1; no longer J3.L, Q2.G, Q3.D, R4.1, U13.1
- net VDD_USB: now also C20.1, D1.A, R1.2, U11.VIN, U2.VOUT; no longer C89.1, C90.1, J13.2, R36.1, R5.1, U11.MODE, U11.VIN1, U16.VDD, U28.IN1
- net VDD_USB_IN: now also J4.1; no longer J13.1
Other:
- note added: ""Separate AGND and PGND. Do not connect AGND and PGND directly at the IC." "Connect AGND and PGND through a via at a different layer.""
- note added: "Capacitor helps minimize reverse current spikes when battery is inserted with reverse polarity."
- note added: "Ceff = 1uF @ 5.5V bias"
- note added: "From "MSP430TM 32-kHz Crystal Oscillators", section "Effective Load Capacitance": Crystal capacitor values are calculated using: C_L = (C + C_para) / 2 Where: C_L = load capacitance from crystal datasheet C = capacitor value to solve for C_para = parasitic capacitance of MSP pin + trace C_para = 2pF (MSP capacitance per pin) + 1 pF (estimated trace capacitance) = 3 pF C_L = 6 pF (from crystal dat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"
- note added: "Limits inrush current and ESD into the gates of our PFETs. (Using 3k instead of 1k to consolidate resistor values.)"
- note added: "Limits the drive strength to limit inrush current and dampen ringing on the PFET's gate. (Using 3k instead of 1k to consolidate resistor values.)"
- note added: "Pull-down is sized so that: - Battery mode: it's much less than the gate leakage resistance of the PFETs, which is about 50 Meg ohms, so that VDD_USB isn't pulled high by the leakage (which would cause USB mode to be erronously enabled.) - USB mode: it doesn't draw too much current"
- note added: "Requirements: - 1% - TCR <= ±200 ppm/°C"
- note added: "STM32's VDDUSB is supposed to rise after its VDD"
- note added: "Schottky Diode requirements: - Low reverse leakage (minimize battery power loss, since battery will reverse bias) - Low forward voltage"
- note added: "This PFET serves 2 purposes for the battery power supply: 1. Provides reverse polarity protection When battery terminals are reversed: - USB disconnected: g=0 & s=0 => Vsg=0 => transistor off, OR - USB connected: g=5 & s=5 => Vsg=0 => transistor off 2. Provides reverse current protection By pulling gate up when USB is connected, voltages > VDD_BAT are blocked from reaching the battery."
- note added: "This buffer blocks the clock while the PIX domain isn't powered. It works simply by taking advantage of the buffer's "I_Off" behavior, which guarantees no leakage between input and output when its VDD=0."
- note added: "Using load switch purely for its soft-start behavior, to limit USB inrush current"
- note added: "VDD_1V2"
- note added: "VDD_1V9"
- note added: "VDD_1V9_IMG"
- note added: "VDD_1V9_STM - Battery: VDD_1V9_STM = HiZ - USB: VDD_1V9_STM = VDD_1V9"
- note added: "VDD_2V8"
- note added: "VDD_2V8_IMG"
- note added: "VDD_2V8_SD"
- note added: "VDD_3V3_STM - Battery: VDD_3V3_STM = HiZ - USB: VDD_3V3_STM = 3V3"
- note added: "VDD_A - Battery: VDD_A = VDD_BAT - USB: VDD_A = 1V9"
- note added: "VDD_B - Battery: VDD_B = HiZ / VDD_BAT (controlled by MSP via !VDD_B_EN!) - USB: VDD_B = VDD_USB"
- note added: "We're using 1.9V instead of 1.8V purely to help meet the Vih of the SD card when it's in 3.3V mode. In 3.3V mode, the SD card is supposed to be supplied 3.3V signals, but the ICE40 gives it 1.9V signals instead. We're doing this because we haven't found a good method of switching the signal voltage without introducing capacitance on the signalling lines (which can greatly impact the 100MHz high-s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"
- note removed: "5.1k resistor requirements: - Tolerance = 10% (20% is acceptable, but 10% is required if, in the future, we want to sense the source's current capability (by reading the voltage on CC1/CC2), to potentially draw more than 500mA if the source supports it.)"
- note removed: "Battery Charge Level"
- note removed: "Battery Charging"
- note removed: "Battery reverse polarity protection"
- note removed: "Capacitance must be limited because it's attached to VDD_USB, which can have a max of 10uF (per USB spec)."
- note removed: "Don't use a pullup resistor on MSP_RST_!! MSP430FR* has an internal 20k-50k pullup, which is already on the low end for correct operation of the level shifter, which requires weak pullups. Adding an external resistor lowers the pullup resistance further (parallel resistors), worsening the level shifter's VOL."
- note removed: "Don't use the recommended 1nF capacitor!! For correct operation of the level shifter, we need a much lower capacitance on MSP_RST, because the level shifter can't drive large capacitive loads. Since the recommended 1nF capacitor is for noise suppression, we should be able to get away with a smaller capacitor."
- note removed: "ESD protection for MOSFETs Requirements: - low reverse leakage current: <= 100nA since this current will be lost when battery powered - reverse working voltage ~= 5V since battery will operate up to ~4.2V"
- note removed: "From "MSP430TM 32-kHz Crystal Oscillators", section "Effective Load Capacitance": Crystal capacitor values are calculated using: C_L = (C + C_para) / 2 Where: C_L = load capacitance from crystal datasheet C = capacitor value to solve for C_para = parasitic capacitance of MSP pin + trace C_para = 2pF (MSP capacitance per pin) + 1 pF (estimated trace capacitance) = 3 pF C_L = 12.5 pF (from crystal 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"
- note removed: "From Linear Tech Application Note 171"
- note removed: "From W25Q40EWUXIE datasheet: "Note that the chip select pin (/CS) must track the VCC supply level at power-up until the VCC-min level and tVSL time delay is reached. If needed a pull-up resister on /CS can be used to accomplish this." We accomplish this because ICE40 has an internal pullup on its SPI_SS_B, which is connected to ICE_ST_SPI_CS_, so the output of the OR gate should be a high voltage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"
- note removed: "Limits drive strength to dampen ringing on the PFET's gate"
- note removed: "NOR gate ensures that VDD_B is unconditionally powered in USB mode"
- note removed: "Pulldown ensures that VDD_USB can be safely used as a binary signal"
- note removed: "Resistor sets battery charge current: I = 1000 / R I = 1000 / 2.7k I = 370 mA"
- note removed: "STM32's VDDUSB is supposed to rise after its VDD (VDD_1V8_STM)"
- note removed: "Schottky diode prevents reverse current through LDO when battery is disconnected. (When the battery is disconnected, it could be the case that the LDO's VOUT > VIN, causing reverse current.) Diode requirements: - Low Vf (forward voltage) so that it activates on a small VOUT-VIN delta - Ir (reverse leakage) < 1µA to minimize leakage when in battery-mode, since this leakage will be constant"
- note removed: "The MOSFET prevents the battery drain caused by the voltage divider until the time comes that we actually need to measure the battery voltage. When we actually want to sample BAT_CHRG_LVL and accept the ensuing battery drain, STM32 asserts BAT_CHRG_LVL_EN_. STM32 is only running when we're connected to USB and therefore charging the battery, in which case we're not concerned with the small amount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"
- note removed: "This buffer blocks the clock while the IMG domain isn't powered. It works simply by taking advantage of the buffer's "I_Off" behavior, which guarantees no leakage between input and output when its VDD=0."
- note removed: "Use VCCB side for VDD_A because VCCB has a wider supply voltage range (1.65-5.5 V), giving us more flexibility in the battery voltage."
- note removed: "VDD_A"
- note removed: "VDD_B"
- note removed: "VDD_B Control"
- note removed: "VDD_B_1V2"
- note removed: "VDD_B_1V8"
- note removed: "VDD_B_1V8_IMG"
- note removed: "VDD_B_1V8_STM - Battery: VDD_B_1V8_STM = HiZ - USB: VDD_B_1V8_STM = VDD_B_1V8"
- note removed: "VDD_B_2V8"
- note removed: "VDD_B_2V8_IMG"
- note removed: "VDD_B_2V8_SD"
- note removed: "VDD_B_3V3_STM - Battery: VDD_B_3V3_STM = HiZ - USB: VDD_B_3V3_STM = VDD_A_3V3"
- note removed: "Voltage divider sets VIN2 -> VIN1 switch voltage to 4V. That is, when VDD_USB reaches 4V, PR1=1V=VREF, so TPS2116 switches its VOUT to be sourced by VDD_USB."
- note removed: "≤ 1% ≤ 200 ppm/°C"
- moved on the sheet: C10, C15, C16, C17, C18, C19, C2, C20, C26, C29, C3, C30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
